File: sound.kicad_sch (KiCad schematic)
At the start: 79 parts

Commit message: Upgrade
Parts:
- added C42, C47: C, 22 pF, symbol PCM_Generic:C,IEC
- added C43, C44, C48: C, 820 pF, symbol PCM_Generic:C,IEC
- added C45, C49, C50: C, 220 pF, symbol PCM_Generic:C,IEC
- added C46: C,680nF, symbol PCM_Generic:C,IEC
- added R31, R33, R34, R36, R37: R, 1 Om, symbol PCM_Generic:R,IEC
- added R32, R35, R38: R,2 Om, symbol PCM_Generic:R,IEC
- added R39: R,1 Om, symbol PCM_Generic:R,IEC
- C12, C16: value C, 22 pF -> C, 220 pF
- C15: value C, 22 pF -> C, 820 pF
- C2: value C,680nF -> C, 22 pF
- C31, C32: value C,10nF -> C,8.2nF
- C7, C9: value C, 100 nF -> C, 680 nF
- R10, R9: value R, 10 Om -> R, 2 Om
- R13, R14: value R, 90 Om -> R, 1 Om
- R15: value R, 10 Om -> R, 1 Om
- R16: value R, 10 Om -> R,2 Om
- R18: value R,5 Om -> R,1Om
- R19, R20, R21, R24, R26, R27: value R,10 Om -> R,2 Om
- R23, R30: value R,5 Om -> R,1 Om
Connections:
- net E: now also R39.2 (-)
- net GNDA: now also C46.2 (-), C50.1 (+), R31.1 (+), R32.1 (+), R33.1 (+), R34.2 (-), R35.1 (+); no longer C2.2 (-), R14.2 (-), R15.2 (-), R16.2 (-)
- net at R14.1 (+): now also C11.2 (-), C17.1 (+), C19.1 (+), C3.1 (+), C31.1 (+), L3.2 (-), R15.2 (-), R16.1 (+), R25.2 (-), R5.2 (-), R6.2 (-), R9.2 (-); no longer C14.1 (+)
- net at C13.2 (-), C5.1 (+), L4.2 (-)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: now also R36.1 (+), R37.2 (-), R38.1 (+); no longer C14.2 (-), C16.1 (+), C18.2 (-), C20.2 (-), C32.2 (-), R25.1 (+)
- net at C2.1 (+), L2.1 (+), R2.1 (+): now also C44.1 (+), C45.2 (-), C46.1 (+)
- net at C15.2 (-): now also R16.2 (-); no longer R15.1 (+)
- net at C9.1 (+), R8.1 (+): now also C18.2 (-), C20.2 (-), C32.2 (-), R25.1 (+)
- net at C16.2 (-): now also C11.1 (+), C14.1 (+), C15.1 (+), L3.1 (+), R11.1 (+); no longer R16.1 (+)
- net at C1.1 (+), L1.1 (+), R1.1 (+): now also C12.2 (-), C42.1 (+), C43.1 (+)
- net at C13.1 (+), L4.1 (+), R12.1 (+): now also C47.1 (+), C48.1 (+), C49.2 (-)
- new net: C48.2 (-), R38.2 (-)
- new net: C47.2 (-), R36.2 (-)
- new net: C43.2 (-), R32.2 (-)
- new net: C2.2 (-), R33.2 (-)
- new net: C50.2 (-), R39.1 (+)
- new net: C42.2 (-), R31.2 (-)
- new net: C14.2 (-), R14.2 (-)
- new net: C45.1 (+), R34.1 (+)
- new net: C16.1 (+), R15.1 (+)
- new net: C44.2 (-), R35.2 (-)
- new net: C49.1 (+), R37.1 (+)
Other:
- moved on the sheet: C13, L1, L3
